File: documentation.kicad_sch (KiCad schematic)
At the start: 0 parts

Commit message: copy_first
Other:
- note added: "BACK"
- note added: "FRONT"
Changed lines of the file:
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@@
 	(generator_version "9.0")
 	(paper "A4")
+	(text "BACK"
+		(exclude_from_sim no)
+		(at 207.01 66.04 0)
+		(effects
+			(font
+				(size 1.27 1.27)
+			)
+		)
+	)
+	(text "FRONT\n"
+		(exclude_from_sim no)
+		(at 92.71 66.04 0)
+		(effects
+			(font
+				(size 1.27 1.27)
+			)
+		)
+	)
 )
